File: psi3214_dispositivo.kicad_pcb (KiCad board)
At the start: 2 copper layers, 83 x 60.5 mm, 13 parts, among them J1 Screw_Terminal_01x02, J2 Screw_Terminal_01x03, U1 TL072_sim

Commit message: PCB with ground plane version
Parts:
- moved R8 56.5 mm to (155.5, 65.5), turned to 90 degrees
- moved R9 55.9 mm to (159.5, 75.5), turned to 90 degrees
- moved C3 54.9 mm to (155.5, 60.5), turned to -90 degrees
- moved R5 50.3 mm to (166.5, 43.5), turned to -90 degrees
- moved R13 49.5 mm to (163.0, 75.5), turned to -90 degrees
- moved C2 44.9 mm to (150.0, 47.0)
- moved R4 44.8 mm to (156.0, 43.0), turned to -90 degrees
- moved U1 41.8 mm to (163.0, 60.0), turned to -90 degrees
- moved R11 41.6 mm to (163.0, 69.0), turned to 90 degrees
- moved J2 41.5 mm to (140.0, 67.4), turned to -90 degrees
- moved R7 41.0 mm to (169.0, 60.0), turned to -90 degrees
- moved R6 40.5 mm to (169.0, 52.0), turned to 90 degrees
- moved J1 0.67 mm to (140.0, 42.0)
Routing:
- net +9V: track 0.00 -> 49.3 mm
- net GND: track 130.4 -> 83.4 mm
- net -9V: track 0.00 -> 25.3 mm
- net /saida_cap: track 0.00 -> 20.8 mm
- net /saida_amp1: track 0.00 -> 20.3 mm
- net Net-(U1B--): track 0.00 -> 15.5 mm
- net /saida_filtro: track 0.00 -> 15.2 mm
- net /saida: track 0.00 -> 12.6 mm
- net Net-(U1A--): track 0.00 -> 9.21 mm
- net /entrada: track 0.00 -> 8.54 mm
Other:
- board size 83 x 60.5 mm -> 39 x 44 mm

Commit message: PCB with no ground plane version
Routing:
- net GND: track 83.4 -> 59.8 mm, vias 5 -> 0
Changed lines of the file:
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@@
 		(layer "Edge.Cuts")
 	)
-	(via
-		(at 166.5 42.0375)
-		(size 1.3)
-		(drill 1)
-		(layers "F.Cu" "B.Cu")
-		(net "GND")
-	)
-	(via
-		(at 155.5 67)
-		(size 1.3)
-		(drill 1)
-		(layers "F.Cu" "B.Cu")
-		(net "GND")
-	)
-	(via
-		(at 159.5 76.9625)
-		(size 1.3)
-		(drill 1)
-		(layers "F.Cu" "B.Cu")
-		(net "GND")
-	)
-	(via
-		(at 156 41.5375)
-		(size 1.3)
-		(drill 1)
-		(layers "F.Cu" "B.Cu")
-		(net "GND")
-	)
-	(via
-		(at 163 76.9625)
-		(size 1.3)
-		(drill 1)
-		(layers "F.Cu" "B.Cu")
-		(net "GND")
-	)
-	(segment
-		(start 166.5 42.0375)
-		(end 156.5 42.0375)
-		(width 1)
-		(layer "B.Cu")
+	(segment
+		(start 166.0375 41.575)
+		(end 166.5 42.0375)
+		(width 1)
+		(layer "F.Cu")
+		(net "GND")
+	)
+	(segment
+		(start 159.5 76.9625)
+		(end 163 76.9625)
+		(width 1)
+		(layer "F.Cu")
 		(net "GND")
 	)
 	(segment
 		(start 155.5 72.9625)
-		(end 155.0325 72.495)
-		(width 1)
-		(layer "B.Cu")
-		(net "GND")
-	)
-	(segment
-		(start 156.5 42.0375)
-		(end 156 41.5375)
-		(width 1)
-		(layer "B.Cu")
+		(end 159.5 76.9625)
+		(width 1)
+		(layer "F.Cu")
+		(net "GND")
+	)
+	(segment
+		(start 145.5325 66.9625)
+		(end 155.5 66.9625)
+		(width 1)
+		(layer "F.Cu")
+		(net "GND")
+	)
+	(segment
+		(start 140 72.495)
+		(end 145.5325 66.9625)
+		(width 1)
+		(layer "F.Cu")
+		(net "GND")
+	)
+	(segment
+		(start 156 41.575)
+		(end 166.0375 41.575)
+		(width 1)
+		(layer "F.Cu")
+		(net "GND")
+	)
+	(segment
+		(start 140 41.955)
+		(end 155.5825 41.955)
+		(width 1)
+		(layer "F.Cu")
 		(net "GND")
 	)
@@
 		(end 155.5 72.9625)
 		(width 1)
-		(layer "B.Cu")
-		(net "GND")
-	)
-	(segment
-		(start 156 41.5375)
-		(end 156 66.5)
-		(width 1)
-		(layer "B.Cu")
-		(net "GND")
-	)
-	(segment
-		(start 140 41.955)
-		(end 155.5825 41.955)
-		(width 1)
-		(layer "B.Cu")
-		(net "GND")
-	)
-	(segment
-		(start 159.5 76.9625)
-		(end 163 76.9625)
-		(width 1)
-		(layer "B.Cu")
-		(net "GND")
-	)
-	(segment
-		(start 155.0325 72.495)
-		(end 140 72.495)
-		(width 1)
-		(layer "B.Cu")
-		(net "GND")
-	)
-	(segment
-		(start 156 66.5)
-		(end 155.5 67)
-		(width 1)
-		(layer "B.Cu")
-		(net "GND")
-	)
-	(segment
-		(start 155.5 72.9625)
-		(end 159.5 76.9625)
-		(width 1)
-		(layer "B.Cu")
+		(layer "F.Cu")
 		(net "GND")
 	)
@@
 		(end 156 41.5375)
 		(width 1)
-		(layer "B.Cu")
+		(layer "F.Cu")
 		(net "GND")
 	)
@@
 		(net "/saida_filtro")
 	)
-	(group ""
-		(members "b1df31cf-611b-4eae-8f1b-b184198d0b5f" "cf0c6875-6bb5-465d-8c63-668fb2609e20")
-	)
-	(group ""
-		(members "52ca1fb2-2743-4492-88dc-2c01721e53fa" "76c002b8-586e-4d77-bfe2-b6e07dbd9fc1")
-	)
-	(group ""
-		(members "4dad2275-4af5-4325-a9b0-c61de657b02a" "68038879-9c9b-4ffd-a0c6-2e97f2d9adca")
-	)
-	(group ""
-		(members "1d925543-c760-4b4a-8db3-7976a5d6231f" "6b6a2e49-9802-4bbf-9c0b-5cb80cec678a")
-	)
-	(group ""
-		(members "3d4d5abc-6ad2-46e5-b22e-9852bd62343e" "f580d812-a0cb-46a4-9266-2a22df860207")
-	)
 	(embedded_fonts no)
