File: psi3214_dispositivo.kicad_pcb (KiCad board)
At the start: 2 copper layers, 39 x 44 mm, 13 parts, among them J1 Screw_Terminal_01x02, J2 Screw_Terminal_01x03, U1 TL072_sim

Commit message: One side
Routing:
- net GND: track 59.8 -> 92.4 mm
- net Net-(U1A--): track 9.21 -> 15.8 mm
- net /saida_filtro: track 15.2 -> 17.3 mm
Changed lines of the file:
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@@
 		(capping no)
 		(filling no)
+		(zone_defaults)
 		(pcbplotparams
 			(layerselection 0x00000000_00000000_55555555_5755f5ff)
@@
 			(outputformat 1)
 			(mirror no)
-			(drillshape 1)
+			(drillshape 0)
 			(scaleselection 1)
-			(outputdirectory "")
+			(outputdirectory "./")
 		)
 	)
@@
 	)
 	(segment
+		(start 137.45 69.945)
+		(end 140 72.495)
+		(width 0.5)
+		(layer "F.Cu")
+		(net "GND")
+	)
+	(segment
+		(start 140 41.955)
+		(end 137.45 44.505)
+		(width 0.5)
+		(layer "F.Cu")
+		(net "GND")
+	)
+	(segment
 		(start 166.0375 41.575)
 		(end 166.5 42.0375)
@@
 	)
 	(segment
+		(start 137.45 44.505)
+		(end 137.45 69.945)
+		(width 0.5)
+		(layer "F.Cu")
+		(net "GND")
+	)
+	(segment
 		(start 155.5 72.9625)
 		(end 159.5 76.9625)
@@
 	)
 	(segment
+		(start 169 47.4625)
+		(end 169 50.5375)
+		(width 0.5)
+		(layer "F.Cu")
+		(net "Net-(U1A--)")
+	)
+	(segment
 		(start 163.635 57.525)
 		(end 163.635 55.9025)
@@
 	)
 	(segment
+		(start 166.5 44.9625)
+		(end 169 47.4625)
+		(width 0.5)
+		(layer "F.Cu")
+		(net "Net-(U1A--)")
+	)
+	(segment
 		(start 162.365 66.9025)
 		(end 163 67.5375)
@@
 		(width 0.5)
 		(layer "F.Cu")
+		(net "/saida_filtro")
+	)
+	(segment
+		(start 155.5 61.975)
+		(end 155.5 64.0375)
+		(width 0.5)
+		(layer "F.Cu")

Commit message: Comercial components
Parts:
- added R10: 1M, Resistor_SMD:R_1206_3216Metric, F.Cu at (173.0, 56.5)
- added R12: 1.5k, Resistor_SMD:R_1206_3216Metric, F.Cu at (155.5, 70.5)
- added R14: 3.3k, Resistor_SMD:R_1206_3216Metric, F.Cu at (150.5, 70.5)
- R7: value 63.6k -> 68k
- R8: value 2030 -> 1k
- moved R6 3.00 mm to (169.0, 49.0)
- moved R5 2.50 mm to (169.0, 43.5)
Connections:
- R8 pad 1: GND -> Net-(R12-Pad2)
Routing:
- net /saida_filtro: track 17.3 -> 26.3 mm
- net /saida_amp1: track 20.3 -> 27.6 mm
- net Net-(R12-Pad2): track 0.00 -> 7.07 mm
- net GND: track 92.4 -> 87.9 mm
Other:
- board size 39 x 44 mm -> 42 x 44 mm

Commit message: Rodolfo v2.0
Parts:
- added J3: Conn_01x02_Socket, Connector_Wire:SolderWire-0.1sqmm_1x02_P3.6mm_D0.4mm_OD1mm, F.Cu at (147.5, 42.7)
- added J4: Conn_01x03, Connector_Wire:SolderWire-0.1sqmm_1x03_P3.6mm_D0.4mm_OD1mm, F.Cu at (147.5, 68.5)
- added J5: Conn_01x02_Socket, Connector_Wire:SolderWire-0.1sqmm_1x02_P3.6mm_D0.4mm_OD1mm, F.Cu at (174.5, 76.5)
- added J6: Screw_Terminal_01x02, TerminalBlock_Phoenix:TerminalBlock_Phoenix_MKDS-1,5-2-5.08_1x02_P5.08mm_Horizontal, F.Cu at (171.7, 71.0)
- moved R7 17.5 mm to (151.5, 60.5)
- moved R10 15.5 mm to (158.0, 60.5), turned to -90 degrees
- moved C2 1.50 mm to (151.5, 47.0)
- moved C3 0.50 mm to (155.0, 60.5)
Routing:
- net GND: track 87.9 -> 127.0 mm
- net /saida: track 12.6 -> 37.9 mm
- net /saida_filtro: track 26.3 -> 14.4 mm
- net -9V: track 25.3 -> 32.9 mm
- net /saida_cap: track 20.8 -> 18.8 mm
- net /entrada: track 8.54 -> 10.0 mm
Other:
- board size 42 x 44 mm -> 43 x 44 mm

Commit message: Pot added
Parts:
- added H1: MountingHole, MountingHole:MountingHole_3.2mm_M3, F.Cu at (137.5, 43.0)
- added H2: MountingHole, MountingHole:MountingHole_3.2mm_M3, F.Cu at (197.5, 43.0)
- added H3: MountingHole, MountingHole:MountingHole_3.2mm_M3, F.Cu at (137.5, 95.0)
- added H4: MountingHole, MountingHole:MountingHole_3.2mm_M3, F.Cu at (198.0, 95.0)
- added R11: Potentiometer, Potentiometer_THT:Potentiometer_Alps_RK09K_Single_Horizontal, F.Cu at (200.0, 81.5)
- added R6: Potentiometer, Potentiometer_THT:Potentiometer_Alps_RK09K_Single_Horizontal, F.Cu at (200.0, 65.0)
- moved C2 13.5 mm to (162.8, 54.5)
- moved J1 13.5 mm to (151.3, 49.4)
- moved R4 13.5 mm to (167.3, 50.5)
- moved R5 13.5 mm to (180.3, 51.0)
- moved R6 13.5 mm to (180.3, 56.5)
- moved C3 13.5 mm to (166.3, 68.0)
- moved J2 13.5 mm to (151.3, 74.9)
- moved J3 13.5 mm to (158.8, 50.2)
- moved J4 13.5 mm to (158.8, 76.0)
- moved J5 13.5 mm to (185.8, 84.0)
- moved J6 13.5 mm to (183.0, 78.5)
- moved R10 13.5 mm to (169.3, 68.0)
- moved R11 13.5 mm to (174.3, 76.5)
- moved R12 13.5 mm to (166.8, 78.0)
- moved R13 13.5 mm to (174.3, 83.0)
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Other:
- board size 43 x 44 mm -> 72.5 x 64.5 mm

Commit message: Done
Parts:
- removed J1, J6: Screw_Terminal_01x02, TerminalBlock_Phoenix:TerminalBlock_Phoenix_MKDS-1,5-2-5.08_1x02_P5.08mm_Horizontal
- removed J3, J5: Conn_01x02_Socket, Connector_Wire:SolderWire-0.1sqmm_1x02_P3.6mm_D0.4mm_OD1mm
- removed the R11 at (174.3, 76.5)
- removed the R11 at (200.0, 81.5)
- removed the R6 at (200.0, 65.0)
- removed the R6 at (180.3, 56.5)
- added BT1: Battery, Beserrovsky:BatteryHolder_Eagle_12BH611-GR, B.Cu at (150.2, 46.4)
- added BT2: Battery, Beserrovsky:BatteryHolder_Eagle_12BH611-GR, B.Cu at (181.7, 46.4)
- added R11: Potentiometer, Potentiometer_THT:Potentiometer_Alps_RK09K_Single_Horizontal, F.Cu at (209.5, 64.0)
- added R6: Potentiometer, Potentiometer_THT:Potentiometer_Alps_RK09K_Single_Horizontal, F.Cu at (209.5, 80.2)
- J2: value Screw_Terminal_01x03 -> AudioJack3; footprint TerminalBlock_Phoenix:TerminalBlock_Phoenix_MKDS-1,5-3-5.08_1x03_P5.08mm_Horizontal -> Connector_Audio:Jack_3.5mm_CUI_SJ1-3525N_Horizontal
- J4: footprint Connector_Wire:SolderWire-0.1sqmm_1x03_P3.6mm_D0.4mm_OD1mm -> TerminalBlock:TerminalBlock_MaiXu_MX126-5.0-03P_1x03_P5.00mm
- moved J4 52.5 mm to (195.5, 38.5), turned to 180 degrees
- moved J2 45.3 mm to (190.5, 97.5), turned to 0 degrees
- moved R4 42.5 mm to (197.4, 80.5), turned to 180 degrees
- moved C2 41.0 mm to (197.4, 76.5), turned to 180 degrees
- moved R9 34.5 mm to (197.4, 61.0), turned to 180 degrees
- moved R5 27.7 mm to (190.9, 76.5), turned to 0 degrees
- moved R13 27.5 mm to (190.9, 61.0), turned to 180 degrees
- moved R14 24.5 mm to (179.4, 60.9), turned to -90 degrees
- moved R12 24.2 mm to (183.9, 61.0), turned to -90 degrees
- moved U1 20.8 mm to (195.0, 69.0), turned to 90 degrees
- moved R7 19.6 mm to (181.9, 72.0), turned to 90 degrees
- moved R10 17.6 mm to (186.4, 72.0), turned to 90 degrees
- moved R8 16.5 mm to (181.9, 66.5), turned to -90 degrees
- moved H2 12.2 mm to (209.0, 39.0)
- moved C3 11.9 mm to (177.4, 72.0), turned to 90 degrees
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Connections:
- net /saida_amp1 renamed saida_amp1
- net /saida_cap renamed saida_cap
- net /saida_filtro renamed saida_filtro
- C2 pad 1: /entrada -> entrada
- R13 pad 1: /saida -> saida
- U1 pad 7: /saida -> saida
Routing:
- net saida: track 0.00 -> 74.7 mm
- net /saida: track 37.9 -> 0.00 mm
- net +9V: track 48.9 -> 86.4 mm, vias 0 -> 2
- net saida_filtro: track 14.4 -> 39.8 mm
- net saida_amp1: track 27.3 -> 45.5 mm
- net GND: track 127.0 -> 111.5 mm, vias 0 -> 5
- net -9V: track 32.9 -> 46.1 mm, vias 0 -> 2
- net Net-(U1A--): track 15.7 -> 28.8 mm
- net /entrada: track 10.0 -> 0.00 mm
- net saida_cap: track 18.8 -> 9.69 mm
- net Net-(U1B--): track 15.5 -> 22.8 mm
Other:
- board size 72.5 x 64.5 mm -> 82 x 67 mm

Commit message: Done
Parts:
- removed BT2: Battery, Beserrovsky:BatteryHolder_Eagle_12BH611-GR
- added C1: 10u, Capacitor_SMD:C_1206_3216Metric, F.Cu at (147.0, 91.0)
- added C4: 10u, Capacitor_SMD:C_1206_3216Metric, F.Cu at (159.5, 92.5)
- added J5: AudioJack3, Connector_Audio:Jack_3.5mm_CUI_SJ1-3525N_Horizontal, F.Cu at (140.9, 75.0)
- added U2: MAX1044, Package_SO:SOIC-8_3.9x4.9mm_P1.27mm, F.Cu at (153.0, 90.6)
- moved C2 50.9 mm to (161.9, 113.0)
- moved C3 50.9 mm to (141.9, 108.5)
- moved H2 50.9 mm to (173.5, 75.5)
- moved H4 50.9 mm to (173.5, 133.5)
- moved J2 50.9 mm to (155.0, 134.0)
- moved R10 50.9 mm to (150.9, 108.5)
- moved R11 50.9 mm to (174.0, 100.5)
- moved R13 50.9 mm to (155.4, 97.5)
- moved R14 50.9 mm to (143.9, 97.4)
- moved R4 50.9 mm to (161.9, 117.0)
- moved R5 50.9 mm to (155.4, 113.0)
- moved R6 50.9 mm to (174.0, 116.7)
- moved R7 50.9 mm to (146.4, 108.5)
- moved R8 50.9 mm to (146.4, 103.0)
- moved R9 50.9 mm to (161.9, 97.5)
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Routing:
- net entrada: track 0.00 -> 66.4 mm, vias 0 -> 1
- net +9V: track 86.4 -> 59.4 mm
- net -9V: track 46.1 -> 56.4 mm
- net GND: track 111.5 -> 120.3 mm, vias 5 -> 7
- net Net-(U2-CAP+): track 0.00 -> 3.75 mm
- net Net-(U2-CAP-): track 0.00 -> 3.58 mm
Other:
- board size 82 x 67 mm -> 51.5 x 67 mm

Commit message: kinda broken state
Parts:
- moved U1 41.0 mm to (200.5, 107.0), turned to 0 degrees
- moved C2 33.8 mm to (195.5, 109.4), turned to 90 degrees
- moved R4 32.0 mm to (193.0, 109.4), turned to 90 degrees
- moved R13 30.9 mm to (146.0, 127.0), turned to -90 degrees
- moved R5 18.9 mm to (173.0, 120.0), turned to 180 degrees
- moved R9 16.0 mm to (173.0, 86.0)
- moved R12 14.1 mm to (143.0, 110.4)
- moved R14 13.5 mm to (140.5, 110.4)
- moved R8 12.5 mm to (141.5, 114.4), turned to 0 degrees
- moved C4 8.03 mm to (152.0, 95.3), turned to 180 degrees
- moved C3 7.83 mm to (147.0, 114.5), turned to 180 degrees
- moved R10 4.10 mm to (147.0, 109.5), turned to 180 degrees
- moved R7 3.52 mm to (147.0, 112.0), turned to 180 degrees
- moved BT1 3.16 mm to (144.5, 81.1)
- moved H1 3.16 mm to (129.0, 72.5)
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Routing:
- net GND: track 120.3 -> 17.5 mm, vias 7 -> 6
- net saida: track 74.7 -> 11.4 mm, vias 0 -> 1
- net entrada: track 66.4 -> 11.4 mm
- net -9V: track 56.4 -> 12.9 mm, vias 2 -> 3
- net +9V: track 59.4 -> 16.0 mm
- net saida_amp1: track 45.5 -> 7.54 mm, vias 0 -> 2
- net saida_filtro: track 39.8 -> 8.22 mm, vias 0 -> 2
- net Net-(U1A--): track 28.8 -> 0.00 mm
- net Net-(U1B--): track 22.8 -> 0.00 mm
- net saida_cap: track 9.69 -> 5.76 mm
- net Net-(R12-Pad2): track 7.01 -> 5.30 mm
- net Net-(U2-CAP-): track 3.58 -> 2.56 mm
- net Net-(U2-CAP+): track 3.75 -> 2.73 mm
