File: psi3214_dispositivo.kicad_sch (KiCad schematic)
At the start: 0 parts

Commit message: Breadboard
Parts:
- added C2: 100n, symbol Device:C
- added C3: 10n, symbol Device:C
- added R11: 27k, symbol Device:R
- added R13, R4: 10k, symbol Device:R
- added R3: 50, symbol Device:R
- added R5: 47k, symbol Device:R
- added R6: 100k, symbol Device:R
- added R7: 63.6k, symbol Device:R
- added R8: 2030, symbol Device:R
- added R9: 6.8k, symbol Device:R
- added U1: TL072, symbol Amplifier_Operational:TL072
- added V1: 1 ac=1, symbol Simulation_SPICE:VDC
- added V2, V3: 9, symbol Simulation_SPICE:VDC
Connections:
- new net: R11.2, R9.2, U1.6 (-)
- new net: C2.1, R3.1
- new net: R3.2, V1.1
- new net: C3.1, R6.1, R7.1, U1.1
- new net: C3.2, R7.2, R8.2, U1.5 (+)
- new net: C2.2, R4.2, U1.3 (+)
- new net: R5.2, R6.2, U1.2 (-)
- new net +9V: U1.8 (V+), V2.1
- new net -9V: U1.4 (V-), V3.2
- new net 0: R13.2, R4.1, R5.1, R8.1, R9.1, V1.2, V2.2, V3.1
- new net out_general: R11.1, R13.1, U1.7

Commit message: Spice Sim working
Parts:
- removed U1: TL072, symbol Amplifier_Operational:TL072
- added R1: 0.0001, symbol Device:R
- added U1: TL072_sim, symbol custom:TL072_sim
- C2: value 100n -> 1u
- R11: value 27k -> 22k
- R5: value 47k -> 1k
- R6: value 100k -> 220
- R9: value 6.8k -> 1k
Connections:
- net +9V: now also U1.8 (V+)
- net -9V: now also U1.4 (V-)
- net 0: now also R1.2; no longer R13.2, R4.1, R5.1, R8.1, R9.1, V1.2, V2.2, V3.1
- net at R11.2, R9.2: now also U1.6 (-)
- net entrada: now reaches C2.1, R3.1
- net saida_amp1: now reaches C3.1, R6.1, R7.1
- net saida_amp1: now also U1.1
- net saida_filtro: now reaches C3.2, R7.2, R8.2
- net saida_filtro: now also U1.5 (+)
- net saida_cap: now reaches C2.2, R4.2
- net saida_cap: now also U1.3 (+)
- net at R5.2, R6.2: now also U1.2 (-)
- net out_general renamed saida
- net saida: now also U1.7
- new net GND: R1.1, R13.2, R4.1, R5.1, R8.1, R9.1, V1.2, V2.2, V3.1
Other:
- added sheet Nova-Folha (untitled.kicad_sch)
- note added: "$$A_v = 1 + \frac{R11}{R9}$$"
- note added: "$$A_v = 1 + \frac{R6}{R5}$$"
- note added: "AmpOp não inversor"
- note added: "fc = 16Hz Remove DC"
- moved on the sheet: V2, V3

Commit message: Updating
Parts:
- added J1: Screw_Terminal_01x02, TerminalBlock_Phoenix:TerminalBlock_Phoenix_MKDS-1,5-2-5.08_1x02_P5.08mm_Horizontal, symbol Connector:Screw_Terminal_01x02
- added J2: Screw_Terminal_01x03, TerminalBlock_Phoenix:TerminalBlock_Phoenix_MKDS-1,5-3-5.08_1x03_P5.08mm_Horizontal, symbol Connector:Screw_Terminal_01x03
- C2, C3: footprint (none) -> Capacitor_SMD:C_1206_3216Metric
- R11, R13, R4, R5, R6, R7, R8, R9: footprint (none) -> Resistor_SMD:R_1206_3216Metric
- R3: footprint (none) -> Resistor_SMD:R_1206_3216Metric; now left out of the parts list
- U1: footprint (none) -> Package_SO:SOIC-8_3.9x4.9mm_P1.27mm
- V1, V2, V3: now left out of the parts list
Connections:
- net +9V: now also J2.3 (Pin_3)
- net -9V: now also J2.1 (Pin_1)
- net GND: now also J1.1 (Pin_1), J2.2 (Pin_2)
- net entrada: now also J1.2 (Pin_2)

Commit message: Comercial components
Parts:
- added R10: 1M, Resistor_SMD:R_1206_3216Metric, symbol Device:R
- added R12: 1.5k, Resistor_SMD:R_1206_3216Metric, symbol Device:R
- added R14: 3.3k, Resistor_SMD:R_1206_3216Metric, symbol Device:R
- R7: value 63.6k -> 68k
- R8: value 2030 -> 1k
Connections:
- net GND: now also R12.1, R14.1; no longer R8.1
- net saida_amp1: now also R10.1
- net saida_filtro: now also R10.2
- new net: R12.2, R14.2, R8.1
Other:
- note added: "Req = ~ 63,6k"
- note added: "Req ~ 2,03k"

Commit message: Rodolfo v2.0
Parts:
- added J3, J5: Conn_01x02_Socket, Connector_Wire:SolderWire-0.1sqmm_1x02_P3.6mm_D0.4mm_OD1mm, symbol Connector:Conn_01x02_Socket
- added J4: Conn_01x03, Connector_Wire:SolderWire-0.1sqmm_1x03_P3.6mm_D0.4mm_OD1mm, symbol Connector_Generic:Conn_01x03
- added J6: Screw_Terminal_01x02, TerminalBlock_Phoenix:TerminalBlock_Phoenix_MKDS-1,5-2-5.08_1x02_P5.08mm_Horizontal, symbol Connector:Screw_Terminal_01x02
Connections:
- net +9V: now also J4.3 (Pin_3)
- net -9V: now also J4.1 (Pin_1)
- net GND: now also J3.1 (Pin_1), J4.2 (Pin_2), J5.1 (Pin_1), J6.1 (Pin_1)
- net entrada: now also J3.2 (Pin_2)
- net saida: now also J5.2 (Pin_2), J6.2 (Pin_2)

Commit message: Latest version dump
Other:
- note added: "Falta Potenciometro"
Changed lines of the file:
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@@
+		)
+	)
+	(text "Falta Potenciometro"
+		(exclude_from_sim no)
+		(at 254.762 25.908 0)
+		(effects
+			(font
+				(size 1.27 1.27)
+			)
 		)
 	)

Commit message: Pot added
Parts:
- removed R11: 22k, Resistor_SMD:R_1206_3216Metric, symbol Device:R
- removed R6: 220, Resistor_SMD:R_1206_3216Metric, symbol Device:R
- added H1, H2, H3, H4: MountingHole, MountingHole:MountingHole_3.2mm_M3, symbol Mechanical:MountingHole
- added R11, R6: Potentiometer, Potentiometer_THT:Potentiometer_Alps_RK09K_Single_Horizontal, symbol Simulation_SPICE:Potentiometer
Connections:
- net saida: now also R11.1
- net saida_amp1: now also R6.1
- net at R5.2, U1.2 (-): now also R6.2
- net at R9.2, U1.6 (-): now also R11.2
- no-connect marks 0 -> 2

Commit message: Done
Parts:
- removed C2: 1u, Capacitor_SMD:C_1206_3216Metric, symbol Device:C
- removed C3: 10n, Capacitor_SMD:C_1206_3216Metric, symbol Device:C
- removed H1, H2, H3, H4: MountingHole, MountingHole:MountingHole_3.2mm_M3, symbol Mechanical:MountingHole
- removed J1, J6: Screw_Terminal_01x02, TerminalBlock_Phoenix:TerminalBlock_Phoenix_MKDS-1,5-2-5.08_1x02_P5.08mm_Horizontal, symbol Connector:Screw_Terminal_01x02
- removed J2: Screw_Terminal_01x03, TerminalBlock_Phoenix:TerminalBlock_Phoenix_MKDS-1,5-3-5.08_1x03_P5.08mm_Horizontal, symbol Connector:Screw_Terminal_01x03
- removed J3, J5: Conn_01x02_Socket, Connector_Wire:SolderWire-0.1sqmm_1x02_P3.6mm_D0.4mm_OD1mm, symbol Connector:Conn_01x02_Socket
- removed J4: Conn_01x03, Connector_Wire:SolderWire-0.1sqmm_1x03_P3.6mm_D0.4mm_OD1mm, symbol Connector_Generic:Conn_01x03
- removed R1: 0.0001, symbol Device:R
- removed R10: 1M, Resistor_SMD:R_1206_3216Metric, symbol Device:R
- removed R11, R6: Potentiometer, Potentiometer_THT:Potentiometer_Alps_RK09K_Single_Horizontal, symbol Simulation_SPICE:Potentiometer
- removed R12: 1.5k, Resistor_SMD:R_1206_3216Metric, symbol Device:R
- removed R13, R4: 10k, Resistor_SMD:R_1206_3216Metric, symbol Device:R
- removed R14: 3.3k, Resistor_SMD:R_1206_3216Metric, symbol Device:R
- removed R3: 50, Resistor_SMD:R_1206_3216Metric, symbol Device:R
- removed R5, R8, R9: 1k, Resistor_SMD:R_1206_3216Metric, symbol Device:R
- removed R7: 68k, Resistor_SMD:R_1206_3216Metric, symbol Device:R
- removed U1: TL072_sim, Package_SO:SOIC-8_3.9x4.9mm_P1.27mm, symbol custom:TL072_sim
- removed V1: 1 ac=1, symbol Simulation_SPICE:VDC
- removed V2, V3: 9, symbol Simulation_SPICE:VDC
Connections:
- no-connect marks 2 -> 0
Other:
- removed sheet Nova-Folha
- added sheet Analogico (untitled.kicad_sch)
- added sheet Conectores e Outros (connectors.kicad_sch)
- note removed: "$$A_v = 1 + \frac{R11}{R9}$$"
- note removed: "$$A_v = 1 + \frac{R6}{R5}$$"
- note removed: "AmpOp não inversor"
- note removed: "Falta Potenciometro"
- note removed: "Req = ~ 63,6k"
- note removed: "Req ~ 2,03k"
- note removed: "fc = 16Hz Remove DC"
