File: untitled.kicad_sch (KiCad schematic)
At the start: 0 parts

Commit message: Done
Parts:
- added C2: 1u, Capacitor_SMD:C_1206_3216Metric, symbol Device:C
- added C3: 10n, Capacitor_SMD:C_1206_3216Metric, symbol Device:C
- added R1: 0.0001, symbol Device:R
- added R10: 1M, Resistor_SMD:R_1206_3216Metric, symbol Device:R
- added R11, R6: Potentiometer, Potentiometer_THT:Potentiometer_Alps_RK09K_Single_Horizontal, symbol Simulation_SPICE:Potentiometer
- added R12: 1.5k, Resistor_SMD:R_1206_3216Metric, symbol Device:R
- added R13, R4: 10k, Resistor_SMD:R_1206_3216Metric, symbol Device:R
- added R14: 3.3k, Resistor_SMD:R_1206_3216Metric, symbol Device:R
- added R3: 50, Resistor_SMD:R_1206_3216Metric, symbol Device:R
- added R5, R8, R9: 1k, Resistor_SMD:R_1206_3216Metric, symbol Device:R
- added R7: 68k, Resistor_SMD:R_1206_3216Metric, symbol Device:R
- added U1: TL072_sim, Package_SO:SOIC-8_3.9x4.9mm_P1.27mm, symbol custom:TL072_sim
- added V1: 1 ac=1, symbol Simulation_SPICE:VDC
- added V2, V3: 9, symbol Simulation_SPICE:VDC
Connections:
- new net: R12.2, R14.2, R8.1
- new net: R5.2, R6.2, U1.2 (-)
- new net: R11.2, R9.2, U1.6 (-)
- new net: R3.2, V1.1
- new net +9V: U1.8 (V+), V2.1
- new net -9V: U1.4 (V-), V3.2
- new net 0: R1.2
- new net GND: R1.1, R12.1, R13.2, R14.1, R4.1, R5.1, R9.1, V1.2, V2.2, V3.1
- new net entrada: C2.1, R3.1
- new net saida: R11.1, R13.1, U1.7
- new net saida_amp1: C3.1, R10.1, R6.1, R7.1, U1.1
- new net saida_cap: C2.2, R4.2, U1.3 (+)
- new net saida_filtro: C3.2, R10.2, R7.2, R8.2, U1.5 (+)
- no-connect marks 0 -> 2
Other:
- note added: "$$A_v = 1 + \frac{R11}{R9}$$"
- note added: "$$A_v = 1 + \frac{R6}{R5}$$"
- note added: "AmpOp não inversor"
- note added: "Req = ~ 63,6k"
- note added: "Req ~ 2,03k"
- note added: "fc = 16Hz Remove DC"
